Commit message: starting to look amazing

File: eric-personal-website/src/assets/urdf/simple_3dof.urdf (robot description, URDF)
Before this commit: robot simple_3dof, 6 links, 5 joints
Joints:
- joint ee_joint: origin xyz=0.2 0.0 0.0 rpy=0.0 0.0 0.0 -> xyz=0.1 0.0 0.0 rpy=0.0 0.0 0.0
- joint joint1: limit lower=-3.14159 upper=3.14159 effort=30 velocity=2.0 -> lower=-0.7854 upper=0.7854 effort=30 velocity=2.0; origin xyz=0.0 0.0 0.1 rpy=0.0 0.0 0.0 -> xyz=0.0 0.0 0.0 rpy=0.0 0.0 0.0
- joint joint2: limit lower=-3.14159 upper=3.14159 effort=30 velocity=2.0 -> lower=-0.3927 upper=1.5708 effort=30 velocity=2.0; origin xyz=0.3 0.0 0.0 rpy=0.0 1.5708 0.0 -> xyz=0.0 0.0 0.0 rpy=0.0 1.5708 0.0
- joint joint3: limit lower=-3.14159 upper=3.14159 effort=30 velocity=2.0 -> lower=0. upper=1.5708 effort=30 velocity=2.0; origin xyz=0.3 0.0 0.0 rpy=0.0 0.0 0.0 -> xyz=0.2 0.0 0.0 rpy=0.0 0.0 0.0
