Commit message: this is looking crazy good

File: eric-personal-website/src/assets/urdf/simple_3dof_f_a_f.urdf (robot description, URDF)
Before this commit: robot simple_3dof, 6 links, 5 joints
Joints:
- joint ee_joint: origin xyz=0.1 0.0 0.0 rpy=0.0 0.0 0.0 -> xyz=0.0 0.4 0.0 rpy=0.0 0.0 0.0
- joint joint1: axis 0 0 1 -> 1 0 0; limit lower=-0.7854 upper=0.7854 effort=30 velocity=2.0 -> lower=-1.5708 upper=0.0 effort=30 velocity=2.0
- joint joint2: limit lower=-0.3927 upper=1.5708 effort=30 velocity=2.0 -> lower=-0.7854 upper=0.7854 effort=30 velocity=2.0; origin xyz=0.0 0.0 0.0 rpy=0.0 1.5708 0.0 -> xyz=0.0 0.0 0.0 rpy=0.0 0.0 0.0
- joint joint3: axis 0 0 1 -> 1 0 0; limit lower=0. upper=1.5708 effort=30 velocity=2.0 -> lower=-1.5708 upper=0.0 effort=30 velocity=2.0; origin xyz=0.2 0.0 0.0 rpy=0.0 0.0 0.0 -> xyz=0.0 0.4 0.0 rpy=0.0 0.0 0.0
