Commit message: final changes

File: eric-personal-website/src/assets/urdf/shoulder_3r.urdf (robot description, URDF)
Before this commit: robot shoulder_3r, 6 links, 5 joints
Joints:
- joint joint2: origin xyz=0.0 0.0 0.0 rpy=0.0 0.0 0.0 -> xyz=0.0 0.0 0.08 rpy=0.0 0.0 0.0
- joint joint3: axis 1 0 0 -> 0 0 1; origin xyz=0.0 0.0 0.0 rpy=0.0 0.0 0.0 -> xyz=0.0 0.0 0.08 rpy=0.0 0.0 0.0
